Commit message: Modify USD acquisition method to use template-based configuration

File: example/pick_place_agilebot_camera_gripper/rmpflow/gbt-c5a_camera_gripper.urdf (robot description, URDF)
Before this commit: robot GBT_C5A, 25 links, 24 joints
Links:
- removed link Orbbec
- removed link base_link
- removed link camera_mount
- removed link camera_rgb
- removed link camera_tof_nfov
- removed link camera_tof_wfov
- removed link ee_link
- removed link flange
- removed link link1
- removed link link2
- removed link link3
- removed link link4
- removed link link5
- removed link link6
- removed link robotiq_arg2f_base_link
- added link GBT_C5A_wrist_camera_gripper
- added link GBT_C5A_wrist_camera_gripper_base_link, mass 1.489536; collision mesh filename=file:///home/gbt/ws/urdf/gbt-c5a_wrist_camera_gripper/meshe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 scale=1. 1. 1.; visual mesh filename=file:///home/gbt/ws/urdf/gbt-c5a_wrist_camera_gripper/meshe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 scale=1. 1. 1.
- added link GBT_C5A_wrist_camera_gripper_link1, mass 4.7630582; collision mesh filename=file:///home/gbt/ws/urdf/gbt-c5a_wrist_camera_gripper/meshe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 scale=1. 1. 1.; visual mesh filename=file:///home/gbt/ws/urdf/gbt-c5a_wrist_camera_gripper/meshe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 scale=1. 1. 1.
- added link GBT_C5A_wrist_camera_gripper_link2, mass 10.9228296; collision mesh filename=file:///home/gbt/ws/urdf/gbt-c5a_wrist_camera_gripper/meshe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 scale=1. 1. 1.; visual mesh filename=file:///home/gbt/ws/urdf/gbt-c5a_wrist_camera_gripper/meshe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 scale=1. 1. 1.
- added link GBT_C5A_wrist_camera_gripper_link3, mass 3.817807; collision mesh filename=file:///home/gbt/ws/urdf/gbt-c5a_wrist_camera_gripper/meshe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 scale=1. 1. 1.; visual mesh filename=file:///home/gbt/ws/urdf/gbt-c5a_wrist_camera_gripper/meshe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 scale=1. 1. 1.
- added link GBT_C5A_wrist_camera_gripper_link4, mass 1.860492; collision mesh filename=file:///home/gbt/ws/urdf/gbt-c5a_wrist_camera_gripper/meshe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 scale=1. 1. 1.; visual mesh filename=file:///home/gbt/ws/urdf/gbt-c5a_wrist_camera_gripper/meshe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 scale=1. 1. 1.
- added link GBT_C5A_wrist_camera_gripper_link5, mass 1.823601; collision mesh filename=file:///home/gbt/ws/urdf/gbt-c5a_wrist_camera_gripper/meshe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 scale=1. 1. 1.; visual mesh filename=file:///home/gbt/ws/urdf/gbt-c5a_wrist_camera_gripper/meshe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 scale=1. 1. 1.
- added link GBT_C5A_wrist_camera_gripper_link6, mass 0.240531; collision mesh filename=file:///home/gbt/ws/urdf/gbt-c5a_wrist_camera_gripper/meshe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 scale=1. 1. 1.; visual mesh filename=file:///home/gbt/ws/urdf/gbt-c5a_wrist_camera_gripper/meshe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 scale=1. 1. 1.
- added link GBT_C5A_wrist_camera_gripper_robotiq_arg2f_base_link, mass 0.22652; collision mesh filename=file:///home/gbt/ws/urdf/gbt-c5a_wrist_camera_gripper/meshe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 scale=1. 1. 1.; visual mesh filename=file:///home/gbt/ws/urdf/gbt-c5a_wrist_camera_gripper/meshe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 scale=1. 1. 1.
- added link Stream_depth
- added link Stream_depth_OmniverseKitViewportCameraMesh
- added link Stream_ir_left
- added link Stream_ir_left_OmniverseKitViewportCameraMesh
- added link Stream_ir_right
- added link Stream_ir_right_OmniverseKitViewportCameraMesh
- added link Stream_rgb
- added link Stream_rgb_OmniverseKitViewportCameraMesh
- added link camera_link, mass 1.; visual mesh filename=file:///home/gbt/ws/urdf/gbt-c5a_wrist_camera_gripper/meshe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 scale=1. 1. 1.; visual mesh filename=file:///home/gbt/ws/urdf/gbt-c5a_wrist_camera_gripper/meshe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 scale=1. 1. 1.
- added link camera_mount_link, mass 0.16; collision mesh filename=file:///home/gbt/ws/urdf/gbt-c5a_wrist_camera_gripper/meshe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 scale=1. 1. 1.; visual mesh filename=file:///home/gbt/ws/urdf/gbt-c5a_wrist_camera_gripper/meshe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 scale=1. 1. 1.
- added link tcp, mass 1.
- link left_inner_finger: mass 0.0104003125914103 -> 0.0104003; geometry collision mesh filename=file:///home/gbt/ws/urdf/gbt-c5a_wrist_camera_gripper/meshe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 scale=1. 1. 1.; visual mesh filename=file:///home/gbt/ws/urdf/gbt-c5a_wrist_camera_gripper/meshe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 scale=1. 1. 1.
- link left_inner_finger_pad: mass None -> 0.01575; geometry collision box size=0.03 0.07 0.0075; visual box size=0.027 0.065 0.0075
- link left_inner_knuckle: mass 0.0271177346495152 -> 0.0271177; geometry collision mesh filename=file:///home/gbt/ws/urdf/gbt-c5a_wrist_camera_gripper/meshe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 scale=1. 1. 1.; visual mesh filename=file:///home/gbt/ws/urdf/gbt-c5a_wrist_camera_gripper/meshe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 scale=1. 1. 1.
- link left_outer_finger: mass 0.022614240507152 -> 0.0226142; geometry collision mesh filename=file:///home/gbt/ws/urdf/gbt-c5a_wrist_camera_gripper/meshe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 scale=1. 1. 1.; visual mesh filename=file:///home/gbt/ws/urdf/gbt-c5a_wrist_camera_gripper/meshe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 scale=1. 1. 1.
- link left_outer_knuckle: mass 0.00853198276973456 -> 0.008532; geometry collision mesh filename=file:///home/gbt/ws/urdf/gbt-c5a_wrist_camera_gripper/meshe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 scale=1. 1. 1.; visual mesh filename=file:///home/gbt/ws/urdf/gbt-c5a_wrist_camera_gripper/meshe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 scale=1. 1. 1.
- link right_inner_finger: mass 0.0104003125914103 -> 0.0104003; geometry collision mesh filename=file:///home/gbt/ws/urdf/gbt-c5a_wrist_camera_gripper/meshe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 scale=1. 1. 1.; visual mesh filename=file:///home/gbt/ws/urdf/gbt-c5a_wrist_camera_gripper/meshe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 scale=1. 1. 1.
- link right_inner_finger_pad: mass None -> 0.01575; geometry collision box size=0.03 0.07 0.0075; visual box size=0.027 0.065 0.0075
- link right_inner_knuckle: mass 0.0271177346495152 -> 0.0271177; geometry collision mesh filename=file:///home/gbt/ws/urdf/gbt-c5a_wrist_camera_gripper/meshe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 scale=1. 1. 1.; visual mesh filename=file:///home/gbt/ws/urdf/gbt-c5a_wrist_camera_gripper/meshe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 scale=1. 1. 1.
- link right_outer_finger: mass 0.022614240507152 -> 0.0226142; geometry collision mesh filename=file:///home/gbt/ws/urdf/gbt-c5a_wrist_camera_gripper/meshe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 scale=1. 1. 1.; visual mesh filename=file:///home/gbt/ws/urdf/gbt-c5a_wrist_camera_gripper/meshe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 scale=1. 1. 1.
- link right_outer_knuckle: mass 0.00853198276973456 -> 0.008532; geometry collision mesh filename=file:///home/gbt/ws/urdf/gbt-c5a_wrist_camera_gripper/meshe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 scale=1. 1. 1.; visual mesh filename=file:///home/gbt/ws/urdf/gbt-c5a_wrist_camera_gripper/meshe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 scale=1. 1. 1.
Joints:
- removed joint camera_mount_ee_joint
- removed joint camera_mount_orbbec_joint
- removed joint ee_link_root_joint
- removed joint joint_Orbbec-camera_rgb
- removed joint joint_Orbbec-camera_tof_nfov
- removed joint joint_Orbbec-camera_tof_wfov
- removed joint link6_flange
- added joint camera_link_joint: type fixed, parent camera_mount_link, child camera_link, origin xyz=0. 0.01325 -0.06997 rpy=-1.2217307 0. 0. 
- added joint gripper_joint: type fixed, parent camera_mount_link, child GBT_C5A_wrist_camera_gripper_robotiq_arg2f_base_link, origin xyz=0. 0.012 -0.  rpy=3.1415925 -1.5707961 1.5707964
- added joint joint_Stream_depth-viewport_mesh: type fixed, parent Stream_depth, child Stream_depth_OmniverseKitViewportCameraMesh, origin xyz=0. 0. 0. rpy=0. 0. 0.
- added joint joint_Stream_ir_left-viewport_mesh: type fixed, parent Stream_ir_left, child Stream_ir_left_OmniverseKitViewportCameraMesh, origin xyz=0. 0. 0. rpy=0. 0. 0.
- added joint joint_Stream_ir_right-viewport_mesh: type fixed, parent Stream_ir_right, child Stream_ir_right_OmniverseKitViewportCameraMesh, origin xyz=0. 0. 0. rpy=0. 0. 0.
- added joint joint_Stream_rgb-viewport_mesh: type fixed, parent Stream_rgb, child Stream_rgb_OmniverseKitViewportCameraMesh, origin xyz=0. 0. 0. rpy=0. 0. 0.
- added joint joint_camera_link-Stream_depth: type fixed, parent camera_link, child Stream_depth, origin xyz=-0.025 -0. 0.0061397 rpy=-3.1415925 0. -3.1415927
- added joint joint_camera_link-Stream_ir_left: type fixed, parent camera_link, child Stream_ir_left, origin xyz=-0.025 -0. 0.0061397 rpy=-3.1415925 0. -3.1415927
- added joint joint_camera_link-Stream_ir_right: type fixed, parent camera_link, child Stream_ir_right, origin xyz=0.025 -0.0000002 0.0061398 rpy=-3.1415925 0. -3.1415927
- added joint joint_camera_link-Stream_rgb: type fixed, parent camera_link, child Stream_rgb, origin xyz=0.010989 -0.0000077 0.0076121 rpy=-3.1415925 0. -3.1415927
- added joint root_joint: type fixed, parent GBT_C5A_wrist_camera_gripper, child GBT_C5A_wrist_camera_gripper_base_link, origin xyz=0. 0. 0. rpy=0. 0. 0.
- added joint tcp_joint: type fixed, parent GBT_C5A_wrist_camera_gripper_robotiq_arg2f_base_link, child tcp, origin xyz=0. 0. 0.234 rpy=-0.0000001 0.0000001 0.0000002
- joint camera_mount_joint: child camera_mount -> camera_mount_link; origin xyz=0 0 0.003 rpy=0 0 0 -> xyz=0. 0. 0.012 rpy=1.5707965 0. -3.1415925; parent flange -> GBT_C5A_wrist_camera_gripper_link6
- joint finger_joint: axis -1 0 0 -> 1. 0. 0.; limit lower=0 upper=0.7 effort=1000 velocity=2.0 -> lower=0. upper=0.7 effort=1000. velocity=1.9999999; origin xyz=0 -0.030601 0.054905 rpy=2.2957963267948966 0 0 -> xyz=0. -0.030601 0.054905 rpy=-2.2957964 -0.0000001 -3.1415925; parent robotiq_arg2f_base_link -> GBT_C5A_wrist_camera_gripper_robotiq_arg2f_base_link
- joint joint1: axis 0 0 1 -> 0. 0. 1.; child link1 -> GBT_C5A_wrist_camera_gripper_link1; limit lower=-6.283185307179 upper=6.283185307179 effort=100 velocity=1 -> lower=-6.2831853 upper=6.2831853 effort=100. velocity=0.9999999; origin xyz=0 0 0.178 rpy=0 0 0 -> xyz=0. 0. 0.178 rpy=0. 0. 0.; parent base_link -> GBT_C5A_wrist_camera_gripper_base_link
- joint joint2: axis 0 0 1 -> 0. 0. 1.; child link2 -> GBT_C5A_wrist_camera_gripper_link2; limit lower=-1.483529864195 upper=4.625122517784 effort=100 velocity=1 -> lower=-1.4835297 upper=4.6251225 effort=100. velocity=0.9999999; origin xyz=0 0.147 0 rpy=1.5707963267948966 0 0 -> xyz=0. 0.147 0.  rpy=1.5707964 0. 0. ; parent link1 -> GBT_C5A_wrist_camera_gripper_link1
- joint joint3: axis 0 0 1 -> 0. 0. 1.; child link3 -> GBT_C5A_wrist_camera_gripper_link3; limit lower=-2.879793265790 upper=2.879793265790 effort=100 velocity=1 -> lower=-2.879793 upper=2.879793 effort=100. velocity=0.9999999; origin xyz=0.425 0 0.072 rpy=0 0 0 -> xyz=0.425 -0. 0.072 rpy=0. 0. 0.; parent link2 -> GBT_C5A_wrist_camera_gripper_link2
- joint joint4: axis 0 0 1 -> 0. 0. 1.; child link4 -> GBT_C5A_wrist_camera_gripper_link4; limit lower=-1.483529864195 upper=4.625122517784 effort=100 velocity=1 -> lower=-1.4835297 upper=4.6251225 effort=100. velocity=0.9999999; origin xyz=0.385 0 -0.052 rpy=0 0 0 -> xyz=0.385 0. -0.052 rpy=0. 0. 0.; parent link3 -> GBT_C5A_wrist_camera_gripper_link3
- joint joint5: axis 0 0 1 -> 0. 0. 1.; child link5 -> GBT_C5A_wrist_camera_gripper_link5; limit lower=-6.283185307179 upper=6.283185307179 effort=100 velocity=1 -> lower=-6.2831853 upper=6.2831853 effort=100. velocity=0.9999999; origin xyz=0 -0.1233 0 rpy=1.5707963267948966 0 0 -> xyz=-0. -0.1233 0.  rpy=1.5707964 0. 0. ; parent link4 -> GBT_C5A_wrist_camera_gripper_link4
- joint joint6: axis 0 0 1 -> 0. 0. 1.; child link6 -> GBT_C5A_wrist_camera_gripper_link6; limit lower=-6.283185307179 upper=6.283185307179 effort=100 velocity=1 -> lower=-6.2831853 upper=6.2831853 effort=100. velocity=0.9999999; origin xyz=0 -0.1003 0 rpy=1.5707963267948966 0 0 -> xyz=0. -0.1003 -0.  rpy=1.5707963 0. 0. ; parent link5 -> GBT_C5A_wrist_camera_gripper_link5
- joint left_inner_finger_joint: axis 1 0 0 -> 1. 0. 0.; limit lower=-0.8757 upper=0.8757 effort=1000 velocity=2.0 -> lower=-0.14 upper=0.84 effort=0. velocity=17453.2925199; mimic joint=finger_joint multiplier=1 offset=0 -> (none); origin xyz=0 0.0817554015893473 -0.0282203446692936 rpy=-0.725 0 0 -> xyz=-0. 0.0817554 -0.0282204 rpy=-0.725 0. 0. 
- joint left_inner_finger_pad_joint: axis 0 0 1 -> (none); origin xyz=0 0.0457554015893473 -0.0272203446692936 rpy=0 0 0 -> xyz=-0. 0.0457553 -0.0272204 rpy=-0.0000001 -0. -0.0000001
- joint left_inner_knuckle_joint: axis 1 0 0 -> 1. 0. 0.; limit lower=-0.8757 upper=0.8757 effort=1000 velocity=2.0 -> lower=-0.84 upper=0.14 effort=0. velocity=17453.2925199; mimic joint=finger_joint multiplier=-1 offset=0 -> (none); origin xyz=0 -0.0127 0.06142 rpy=2.2957963267948966 0 0.0 -> xyz=0. -0.0127 0.06142 rpy=2.2957964 0.0000001 0.0000002; parent robotiq_arg2f_base_link -> GBT_C5A_wrist_camera_gripper_robotiq_arg2f_base_link
- joint left_outer_finger_joint: axis 1 0 0 -> (none); origin xyz=0 0.01821998610742 0.0260018192872234 rpy=0 0 0 -> xyz=-0. -0.01822 0.0260018 rpy=0.0000002 0.0000002 -3.1415925
- joint right_inner_finger_joint: axis 1 0 0 -> 1. 0. 0.; limit lower=-0.8757 upper=0.8757 effort=1000 velocity=2.0 -> lower=-0.14 upper=0.84 effort=0. velocity=17453.2925199; mimic joint=finger_joint multiplier=1 offset=0 -> (none); origin xyz=0 0.0817554015893473 -0.0282203446692936 rpy=-0.725 0 0 -> xyz=0. 0.0817554 -0.0282204 rpy=-0.725 0. 0. 
- joint right_inner_finger_pad_joint: axis 0 0 1 -> (none); origin xyz=0 0.0457554015893473 -0.0272203446692936 rpy=0 0 0 -> xyz=0. 0.0457553 -0.0272204 rpy=-0.0000001 -0. 0.0000001
- joint right_inner_knuckle_joint: axis 1 0 0 -> 1. 0. 0.; limit lower=-0.8757 upper=0.8757 effort=1000 velocity=2.0 -> lower=-0.84 upper=0.14 effort=0. velocity=17453.2925199; mimic joint=finger_joint multiplier=-1 offset=0 -> (none); origin xyz=0 0.0127 0.06142 rpy=2.2957963267948966 0 -3.141592653589793 -> xyz=0. 0.0127 0.06142 rpy=2.2957966 -0.0000001 -3.1415925; parent robotiq_arg2f_base_link -> GBT_C5A_wrist_camera_gripper_robotiq_arg2f_base_link
- joint right_outer_finger_joint: axis 1 0 0 -> (none); origin xyz=0 0.01821998610742 0.0260018192872234 rpy=0 0 0 -> xyz=-0. 0.0182199 0.0260018 rpy=-0.0000001 -0.0000004 0.0000001
- joint right_outer_knuckle_joint: axis 1 0 0 -> 1. 0. 0.; limit lower=-0.725 upper=0.725 effort=1000 velocity=2.0 -> lower=-0.84 upper=0.14 effort=0. velocity=17453.2925199; mimic joint=finger_joint multiplier=-1 offset=0 -> (none); origin xyz=0 0.030601 0.054905 rpy=2.2957963267948966 0 3.141592653589793 -> xyz=0. 0.030601 0.054905 rpy=2.2957966 -0.0000001 -3.1415925; parent robotiq_arg2f_base_link -> GBT_C5A_wrist_camera_gripper_robotiq_arg2f_base_link
